File: electrolysisMachine/power_distribution.kicad_sch (KiCad schematic)
At the start: 11 parts

Commit message: asdasd
Parts:
- added U2: NE555P, Package_DIP:DIP-8_W7.62mm, symbol Timer:NE555P
Changed lines of the file:
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@@
+	)
+	(symbol
+		(lib_id "Timer:NE555P")
+		(at 156.21 83.82 0)
+		(unit 1)
+		(exclude_from_sim no)
+		(in_bom yes)
+		(on_board yes)
+		(dnp no)
+		(fields_autoplaced yes)
+		(property "Reference" "U2"
+			(at 158.4041 71.12 0)
+			(effects
+				(font
+					(size 1.27 1.27)
+				)
+				(justify left)
+			)
+		)
+		(property "Value" "NE555P"
+			(at 158.4041 73.66 0)
+			(effects
+				(font
+					(size 1.27 1.27)
+				)
+				(justify left)
+			)
+		)
+		(property "Footprint" "Package_DIP:DIP-8_W7.62mm"
+			(at 172.72 93.98 0)
+			(effects
+				(font
+					(size 1.27 1.27)
+				)
+				(hide yes)
+			)
+		)
+		(property "Datasheet" "http://www.ti.com/lit/ds/symlink/ne555.pdf"
+			(at 177.8 93.98 0)
+			(effects
+				(font
+					(size 1.27 1.27)
+				)
+				(hide yes)
+			)
+		)
+		(property "Description" "Precision Timers, 555 compatible,  PDIP-8"
+			(at 156.21 83.82 0)
+			(effects
+				(font
+					(size 1.27 1.27)
+				)
+				(hide yes)
+			)
+		)
+		(pin "5"
+		)
+		(pin "1"
+		)
+		(pin "8"
+		)
+		(pin "4"
+		)
+		(pin "3"
+		)
+		(pin "7"
+		)
+		(pin "2"
+		)
+		(pin "6"
+		)
+		(instances
+			(project "electrolysisMachine"
+				(path "/e63e39d7-6ac0-4ffd-8aa3-1841a4541b55/580159ba-edd3-41e3-abcd-ff933f8f1a26"
+					(reference "U2")
+					(unit 1)
+				)
+			)
+		)
 	)
 	(symbol
